File: arm parts/electronics/PCB's/stepperpcb/stepperpcb.kicad_sch (KiCad schematic)
At the start: 82 parts, among them J1 24Vin -, J10 12Vout -, J11 24Vout -, J12 12V GND, J13 5V GND, J14 24V out, J15 S1 5v GND, J16 S2 5v GND, J17 M2 A2 A1 B1 B2, J18 M1 A2 A1 B1 B2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

Commit message: Added comments for extra description in KiCAD schematic, made io description
Other:
- note added: "15.91kHz f cutoff"
- note added: "Addr: 0x20"
- note added: "Addr: 0x21"
- note added: "Addr: 0x22"
- note added: "Addr: 0x23"
- note added: "Analog IO: analog0 : lpf 16kHz, used as absolute position sens. analog1 : lpf 16kHz, used as absolute position sens. analog2 : directly routed to ardu analog3 : directly routed to ardu (4,5 dont exist) analog6 : directly routed to ardu analog7 : directly routed to ardu"
- note added: "Board I/O cheatsheet: Inputs: J1 : power 24V in J20 analog0 input J6 analog1 input J7 analog 2,3,6,7 + 5V Outputs: J4 servo0 : servo power + signal J15 servo1 : servo power + signal J16 servo2 : servo power + signal J11 : 24V out J9 : 5V out J10 : 12 vout Bidirectional: J2 - I2C (shared with stepper mux's) J5 digital0 : general purpose J21 digial1 : general purpose"
- note added: "U2 is swapped with BUCK module"
- moved on the sheet: J3
Changed lines of the file:
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@@
 (kicad_sch
-	(version 20231120)
+	(version 20250114)
 	(generator "eeschema")
-	(generator_version "8.0")
+	(generator_version "9.0")
 	(paper "A3")
+	(text "15.91kHz f cutoff"
+		(exclude_from_sim no)
+		(at 244.856 50.038 0)
+		(effects
+			(font
+				(size 1.27 1.27)
+			)
+		)
+	)
+	(text "Addr: 0x22\n"
+		(exclude_from_sim no)
+		(at 301.498 173.228 0)
+		(effects
+			(font
+				(size 1.27 1.27)
+			)
+		)
+	)
+	(text "Board I/O cheatsheet:\n\nInputs:\n\nJ1 : power 24V in\n\nJ20 analog0 input\nJ6 analog1 input\nJ7 analog 2,3,6,7 + 5V\n\n\n\nOutputs:\n\n\nJ4 servo0 : servo power + signal\nJ15 servo1 : servo power + signal\nJ16 servo2 : servo power + signal\n\n\nJ11 : 24V out\nJ9 : 5V out \nJ10 : 12 vout\n\n\n\nBidirectional:\n\nJ2 - I2C (shared with stepper mux's)\nJ5 digital0 : general purpose\nJ21 digial1 : general purpose\n"
+		(exclude_from_sim no)
+		(at 181.356 131.064 0)
+		(effects
+			(font
+				(size 1.27 1.27)
+			)
+			(justify left)
+		)
+	)
+	(text "Addr: 0x23\n\n"
+		(exclude_from_sim no)
+		(at 305.308 226.314 0)
+		(effects
+			(font
+				(size 1.27 1.27)
+			)
+		)
+	)
+	(text "15.91kHz f cutoff"
+		(exclude_from_sim no)
+		(at 244.856 24.13 0)
+		(effects
+			(font
+				(size 1.27 1.27)
+			)
+		)
+	)
+	(text "Addr: 0x20"
+		(exclude_from_sim no)
+		(at 307.594 50.038 0)
+		(effects
+			(font
+				(size 1.27 1.27)
+			)
+		)
+	)
+	(text "U2 is swapped with \nBUCK module"
+		(exclude_from_sim no)
+		(at 75.692 18.542 0)
+		(effects
+			(font
+				(size 1.27 1.27)
+				(thickness 0.254)
+				(bold yes)
+			)
+			(justify left)
+		)
+	)
+	(text "Addr: 0x21"
+		(exclude_from_sim no)
+		(at 310.896 110.744 0)
+		(effects
+			(font
+				(size 1.27 1.27)
+			)
+		)
+	)
+	(text "Analog IO:\n\nanalog0 : lpf 16kHz, used as absolute position sens.\nanalog1 : lpf 16kHz, used as absolute position sens.\nanalog2 : directly routed to ardu\nanalog3 : directly routed to ardu\n(4,5 dont exist)\nanalog6 : directly routed to ardu\nanalog7 : directly routed to ardu"
+		(exclude_from_sim no)
+		(at 72.898 112.776 0)
+		(effects
+			(font
+				(size 1.27 1.27)
+			)
+			(justify left)
+		)
+	)
 	(junction
 		(at 58.42 60.96)
@@
 	(wire
 		(pts
-			(xy 68.58 134.62) (xy 72.39 134.62)
+			(xy 68.58 134.62) (xy 85.09 134.62)
 		)
 		(stroke
@@
 	(wire
 		(pts
+			(xy 82.55 140.97) (xy 82.55 139.7)
+		)
+		(stroke
+			(width 0)
+			(type default)
+		)
+	)
+	(wire
+		(pts
 			(xy 356.87 96.52) (xy 354.33 96.52)
 		)
@@
 	(wire
 		(pts
-			(xy 68.58 137.16) (xy 72.39 137.16)
+			(xy 68.58 137.16) (xy 85.09 137.16)
 		)
 		(stroke
@@
 	(wire
 		(pts
-			(xy 72.39 134.62) (xy 72.39 133.35)
-		)
-		(stroke
-			(width 0)
-			(type default)
-		)
-	)
-	(wire
-		(pts
 			(xy 30.48 30.48) (xy 30.48 38.1)
 		)
@@
 	(wire
 		(pts
-			(xy 72.39 137.16) (xy 72.39 135.89)
-		)
-		(stroke
-			(width 0)
-			(type default)
-		)
-	)
-	(wire
-		(pts
 			(xy 41.91 162.56) (xy 43.18 162.56)
 		)
@@
 	(wire
 		(pts
-			(xy 69.85 138.43) (xy 72.39 138.43)
+			(xy 82.55 139.7) (xy 85.09 139.7)
 		)
 		(stroke
@@
 	(symbol
 		(lib_id "Connector:Conn_01x03_Pin")
-		(at 77.47 135.89 180)
+		(at 90.17 137.16 180)
 		(unit 1)
 		(exclude_from_sim no)
@@
 		(fields_autoplaced yes)
 		(property "Reference" "J3"
-			(at 78.74 134.6199 0)
+			(at 91.44 135.8899 0)
 			(effects
 				(font
@@
 		)
 		(property "Value" "GND RX TX"
-			(at 78.74 137.1599 0)
+			(at 91.44 138.4299 0)
 			(effects
 				(font
@@
 		)
 		(property "Footprint" "Connector_PinHeader_2.54mm:PinHeader_1x03_P2.54mm_Vertical"
-			(at 77.47 135.89 0)
+			(at 90.17 137.16 0)
 			(effects
 				(font
@@
 		)
 		(property "Datasheet" "~"
-			(at 77.47 135.89 0)
+			(at 90.17 137.16 0)
 			(effects
 				(font
@@
 		)
 		(property "Description" "Generic connector, single row, 01x03, script generated"
-			(at 77.47 135.89 0)
+			(at 90.17 137.16 0)
 			(effects
 				(font
@@
 		)
 		(property "Value" "PCF8574AP"
-			(at 321.31 48.006 0)
+			(at 329.946 33.02 0)
 			(effects
 				(font
@@
 	(symbol
 		(lib_id "power:GND")
-		(at 69.85 138.43 0)
+		(at 82.55 140.97 0)
 		(unit 1)
 		(exclude_from_sim no)
@@
 		(fields_autoplaced yes)
 		(property "Reference" "#PWR025"
-			(at 69.85 144.78 0)
+			(at 82.55 147.32 0)
 			(effects
 				(font
@@
 		)
 		(property "Value" "GND"
-			(at 69.85 143.51 0)
+			(at 82.55 146.05 0)
 			(effects
 				(font
@@
 		)
 		(property "Footprint" ""
-			(at 69.85 138.43 0)
+			(at 82.55 140.97 0)
 			(effects
 				(font
@@
 		)
 		(property "Datasheet" ""
-			(at 69.85 138.43 0)
+			(at 82.55 140.97 0)
 			(effects
 				(font
@@
 		)
 		(property "Description" "Power symbol creates a global label with name \"GND\" , ground"
-			(at 69.85 138.43 0)
+			(at 82.55 140.97 0)
 			(effects
 				(font
@@
 		)
 	)
+	(embedded_fonts no)
 )
